File: P4_PCB.kicad_pcb (KiCad board)
At the start: 2 copper layers, 25 parts, among them J1 Conn_01x02_Socket, U1 LM324

Commit message: .
Parts:
- moved D5 83.1 mm to (82.5, 117.5)
- moved R14 73.8 mm to (82.5, 92.4)
- moved TH1 53.1 mm to (82.5, 75.0)
- moved C3 47.0 mm to (95.0, 88.0)
- moved R5 47.0 mm to (107.5, 82.4)
- moved D1 43.0 mm to (216.3, 105.0)
- moved R1 43.0 mm to (189.9, 105.0)
- moved D4 39.4 mm to (216.3, 75.0)
- moved R4 39.4 mm to (189.9, 75.0)
- moved J1 34.6 mm to (135.0, 47.5)
- moved R6 28.6 mm to (132.5, 67.4)
- moved R7 28.6 mm to (123.0, 82.7)
- moved C2 26.5 mm to (146.5, 47.5)
- moved R8 26.1 mm to (132.5, 94.4)
- moved R9 26.1 mm to (123.0, 109.6)
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Routing:
- net Net-(U1A-+): track 174.9 -> 0.00 mm
- net Net-(R2-Pad1): track 152.8 -> 0.00 mm
- net Net-(R3-Pad1): track 92.8 -> 0.00 mm
- net Net-(R4-Pad1): track 76.3 -> 0.00 mm
- net Net-(U1B--): track 53.7 -> 0.00 mm
- net Net-(U1A--): track 51.0 -> 0.00 mm
- net Net-(U1C--): track 36.6 -> 0.00 mm
- net Net-(U1D--): track 33.6 -> 0.00 mm
- net Net-(D5-A): track 20.8 -> 0.00 mm
- net Net-(D2-A): track 8.62 -> 0.00 mm
- net Net-(D4-A): track 8.61 -> 0.00 mm
- net Net-(D1-A): track 8.61 -> 0.00 mm
- net Net-(D3-A): track 8.34 -> 0.00 mm
- net (no net): track 0.74 -> 0.00 mm

Commit message: .
Routing:
- net GND: track 0.00 -> 380.2 mm, vias 0 -> 6
- net +5V: track 0.00 -> 254.8 mm
- net Net-(R1-Pad1): track 0.00 -> 129.0 mm
- net Net-(U1A-+): track 0.00 -> 109.1 mm, vias 0 -> 4
- net Net-(R2-Pad1): track 0.00 -> 95.2 mm, vias 0 -> 2
- net Net-(R4-Pad1): track 0.00 -> 66.4 mm
- net Net-(U1D--): track 0.00 -> 63.6 mm, vias 0 -> 2
- net Net-(R3-Pad1): track 0.00 -> 40.7 mm, vias 0 -> 2
- net Net-(U1B--): track 0.00 -> 39.6 mm, vias 0 -> 2
- net Net-(U1C--): track 0.00 -> 39.2 mm, vias 0 -> 4
- net Net-(U1A--): track 0.00 -> 23.3 mm, vias 0 -> 1
- net Net-(D2-A): track 0.00 -> 8.62 mm
- net Net-(D4-A): track 0.00 -> 8.61 mm
- net Net-(D1-A): track 0.00 -> 8.61 mm
- net Net-(D3-A): track 0.00 -> 8.34 mm
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Other:
- board outline added: 168.6 x 89.1 mm
